Commit message: 20241116

File: urdf_basics/urdf/assignment1.xacro (robot description, xacro)
@@ -12,12 +12,15 @@
   </xacro:robot_pedestal_urdf>
   <!-- Robot1 -->
-  <xacro:include filename="$(find ur_description)/urdf/ur10.urdf.xacro"/>
-  <xacro:ur10_robot prefix="robot1_" joint_limited="true"/>
+  <xacro:include filename="$(find urdf_basics)/urdf/robot/ufactory_xarm6.urdf.xacro"/>
+  <xacro:ufactory_xarm6 prefix="robot1_" joint_limited="true"/>
+  <xacro:ufactory_xarm6 prefix="robot2_" joint_limited="true"/>
   <!-- Vacuum Gripper1 -->
   <xacro:include filename="$(find ros_industrial_support)/urdf/vacuum_gripper/vacuum_gripper.urdf.xacro"/>
   <xacro:vacuum_gripper_urdf prefix="vacuum_gripper1_" joint_prefix="vacuum_gripper1_joint"/>
+  <xacro:vacuum_gripper_urdf prefix="vacuum_gripper2_" joint_prefix="vacuum_gripper2_joint"/>
   <!-- bins -->
   <xacro:include filename="$(find ros_industrial_support)/urdf/bin/bin.urdf.xacro"/>
   <xacro:bin_urdf prefix="bin_1_"/>
+  <xacro:bin_urdf prefix="bin_2_"/>
   <!-- Joints -->
   <joint name="world_interface_to_world" type="fixed">
@@ -33,11 +36,11 @@
   <!-- robot1 to pedestal. -->
   <joint name="robot1_to_pedestal" type="fixed">
-  <origin xyz="0 0 0.95" rpy="0 0 0" />
-  <parent link="robot1_pedestal_link" />
-  <child link="robot1_base_link" />
+    <origin xyz="0 0 0.95" rpy="0 0 ${radians(90)}" />
+    <parent link="robot1_pedestal_link" />
+    <child link="robot1_xarm_link" />
   </joint>
   <!-- gripper1 to robot1. -->
   <joint name="gripper1_to_robot1" type="fixed">
-    <parent link="robot1_tool0" />
+    <parent link="robot1_link6" />
     <child link="vacuum_gripper1_base_link" />
   </joint>
@@ -47,4 +50,10 @@
     <child link="bin_1_base_link" />
     <origin xyz="-8.0 -2.2 0" rpy="0 0 0" />
+  </joint>
+  <!-- bin 2 -->
+  <joint name="bin_2_joint" type="fixed">
+    <parent link="world_interface" />
+    <child link="bin_2_base_link" />
+    <origin xyz="2.5 1.8 0" rpy="0 0 0" />
   </joint>
   <link name="robot2_pedestal_link">
@@ -64,20 +73,15 @@
     <child link="robot2_pedestal_link" />
   </joint>
-  <!-- Update the below block for assignment 3 here -->
-  <xacro:include filename="$(find urdf_basics)/urdf/robot/lrmate200ic_macro.xacro"/>
-  <xacro:fanuc_lrmate200ic prefix="robot2_" joint_limited="true"/>
-  <joint name="robot2-robot2_pedestal_joint" type="fixed">
+  <!-- robot2 to pedestal. -->
+  <joint name="robot2_to_pedestal" type="fixed">
+    <origin xyz="0 0 0.6" rpy="0 0 ${radians(180)}" />
     <parent link="robot2_pedestal_link" />
-    <child link="robot2_base_link" />
-    <origin xyz="0 0 0.60" rpy="0 0 ${radians(180)}" />
+    <child link="robot2_xarm_link" />
   </joint>
-<!--
-  <xacro:include filename="$(find ur_description)/urdf/ur5.urdf.xacro"/>
-  <xacro:ur5_robot prefix="robot2_" joint_limited="true"/>
-  <joint name="robot2-robot2_pedestal_joint" type="fixed">
-    <parent link="robot2_pedestal_link" />
-    <child link="robot2_base_link" />
-    <origin xyz="0 0 0.6" rpy="0 0 ${radians(90)}" />
+  <!-- gripper2 to robot1. -->
+  <joint name="gripper2_to_robot2" type="fixed">
+    <parent link="robot2_link6" />
+    <child link="vacuum_gripper2_base_link" />
   </joint>
--->
+  <!-- Add your solution to assignment 1 here -->
 </robot>

File: urdf_basics/urdf/assignment2.xacro (robot description, xacro)
@@ -12,12 +12,15 @@
   </xacro:robot_pedestal_urdf>
   <!-- Robot1 -->
-  <xacro:include filename="$(find ur_description)/urdf/ur10.urdf.xacro"/>
-  <xacro:ur10_robot prefix="robot1_" joint_limited="true"/>
+  <xacro:include filename="$(find urdf_basics)/urdf/robot/ufactory_xarm6.urdf.xacro"/>
+  <xacro:ufactory_xarm6 prefix="robot1_" joint_limited="true"/>
+  <xacro:ufactory_xarm6 prefix="robot2_" joint_limited="true"/>
   <!-- Vacuum Gripper1 -->
   <xacro:include filename="$(find ros_industrial_support)/urdf/vacuum_gripper/vacuum_gripper.urdf.xacro"/>
   <xacro:vacuum_gripper_urdf prefix="vacuum_gripper1_" joint_prefix="vacuum_gripper1_joint"/>
+  <xacro:vacuum_gripper_urdf prefix="vacuum_gripper2_" joint_prefix="vacuum_gripper2_joint"/>
   <!-- bins -->
   <xacro:include filename="$(find ros_industrial_support)/urdf/bin/bin.urdf.xacro"/>
   <xacro:bin_urdf prefix="bin_1_"/>
+  <xacro:bin_urdf prefix="bin_2_"/>
   <!-- Joints -->
   <joint name="world_interface_to_world" type="fixed">
@@ -33,11 +36,11 @@
   <!-- robot1 to pedestal. -->
   <joint name="robot1_to_pedestal" type="fixed">
-  <origin xyz="0 0 0.95" rpy="0 0 0" />
-  <parent link="robot1_pedestal_link" />
-  <child link="robot1_base_link" />
+    <origin xyz="0 0 0.95" rpy="0 0 ${radians(90)}" />
+    <parent link="robot1_pedestal_link" />
+    <child link="robot1_xarm_link" />
   </joint>
   <!-- gripper1 to robot1. -->
   <joint name="gripper1_to_robot1" type="fixed">
-    <parent link="robot1_tool0" />
+    <parent link="robot1_link6" />
     <child link="vacuum_gripper1_base_link" />
   </joint>
@@ -47,4 +50,10 @@
     <child link="bin_1_base_link" />
     <origin xyz="-8.0 -2.2 0" rpy="0 0 0" />
+  </joint>
+  <!-- bin 2 -->
+  <joint name="bin_2_joint" type="fixed">
+    <parent link="world_interface" />
+    <child link="bin_2_base_link" />
+    <origin xyz="2.5 1.8 0" rpy="0 0 0" />
   </joint>
   <link name="robot2_pedestal_link">
@@ -64,28 +73,15 @@
     <child link="robot2_pedestal_link" />
   </joint>
-  <xacro:include filename="$(find ur_description)/urdf/ur5.urdf.xacro"/>
-  <xacro:ur5_robot prefix="robot2_" joint_limited="true"/>
-  <joint name="robot2-robot2_pedestal_joint" type="fixed">
+  <!-- robot2 to pedestal. -->
+  <joint name="robot2_to_pedestal" type="fixed">
+    <origin xyz="0 0 0.6" rpy="0 0 ${radians(180)}" />
     <parent link="robot2_pedestal_link" />
-    <child link="robot2_base_link" />
-    <origin xyz="0 0 0.6" rpy="0 0 ${radians(90)}" />
+    <child link="robot2_xarm_link" />
   </joint>
-  <material name="green">
-    <color rgba="0 1 0 1"/>
-  </material>
-  <link name="sphere">
-    <visual>
-       <geometry>
-         <sphere radius="0.4"/>
-       </geometry>
-       <origin rpy="0 0 0" xyz="0 0 0.4"/>
-       <material name="green"/>
-     </visual>
-   </link>
-   <joint name="world_interface_to_sphere" type="fixed">
-     <parent link="world_interface"/>
-     <child link="sphere"/>
-     <origin xyz="5.5 -5.0 0"/>
-   </joint>
+  <!-- gripper2 to robot1. -->
+  <joint name="gripper2_to_robot2" type="fixed">
+    <parent link="robot2_link6" />
+    <child link="vacuum_gripper2_base_link" />
+  </joint>
   <!-- Add your solution to assignment 2 here -->
 </robot>

File: urdf_basics/urdf/assignment3.xacro (robot description, xacro)
@@ -11,18 +11,13 @@
     <origin xyz="0.5 1.8 0.0" rpy="0 0 0"/>
   </xacro:robot_pedestal_urdf>
-  <!-- Robot1 -->
-  <!--
-  <xacro:include filename="$(find ur_description)/urdf/ur10.urdf.xacro"/>
-  <xacro:ur10_robot prefix="robot1_" joint_limited="true"/>
-  -->
+   <!-- Robot1 -->
+  <xacro:include filename="$(find urdf_basics)/urdf/robot/ufactory_xarm6.urdf.xacro"/>
+  <xacro:ufactory_xarm6 prefix="robot1_" joint_limited="true"/>
   <!-- Vacuum Gripper1 -->
-  <!--
   <xacro:include filename="$(find ros_industrial_support)/urdf/vacuum_gripper/vacuum_gripper.urdf.xacro"/>
   <xacro:vacuum_gripper_urdf prefix="vacuum_gripper1_" joint_prefix="vacuum_gripper1_joint"/>
-  -->
   <!-- bins -->
   <xacro:include filename="$(find ros_industrial_support)/urdf/bin/bin.urdf.xacro"/>
   <xacro:bin_urdf prefix="bin_1_"/>
-  <xacro:bin_urdf prefix="bin_2_"/>
   <!-- Joints -->
   <joint name="world_interface_to_world" type="fixed">
@@ -37,18 +32,14 @@
   </joint>
   <!-- robot1 to pedestal. -->
-  <!--
   <joint name="robot1_to_pedestal" type="fixed">
-  <origin xyz="0 0 0.95" rpy="0 0 0" />
-  <parent link="robot1_pedestal_link" />
-  <child link="robot1_base_link" />
+    <origin xyz="0 0 0.95" rpy="0 0 ${radians(90)}" />
+    <parent link="robot1_pedestal_link" />
+    <child link="robot1_xarm_link" />
   </joint>
-  -->
   <!-- gripper1 to robot1. -->
-  <!--
   <joint name="gripper1_to_robot1" type="fixed">
-    <parent link="robot1_tool0" />
+    <parent link="robot1_link6" />
     <child link="vacuum_gripper1_base_link" />
   </joint>
-  -->
   <!-- bin 1 -->
   <joint name="bin_1_joint" type="fixed">
@@ -56,10 +47,4 @@
     <child link="bin_1_base_link" />
     <origin xyz="-8.0 -2.2 0" rpy="0 0 0" />
-  </joint>
-  <!-- bin 2 -->
-  <joint name="bin_2_joint" type="fixed">
-    <parent link="world_interface" />
-    <child link="bin_2_base_link" />
-    <origin xyz="2.5 1.8 0" rpy="0 0 0" />
   </joint>
   <link name="robot2_pedestal_link">
@@ -79,13 +64,13 @@
     <child link="robot2_pedestal_link" />
   </joint>
+  <!-- Update the below block for assignment 3 here -->
+  <xacro:include filename="$(find urdf_basics)/urdf/robot/lrmate200ic_macro.xacro"/>
+  <xacro:fanuc_lrmate200ic prefix="robot2_"/>
   <!--
-  <xacro:include filename="$(find ur_description)/urdf/ur5.urdf.xacro"/>
-  <xacro:ur5_robot prefix="robot2_" joint_limited="true"/>
-  <joint name="robot2-robot2_pedestal_joint" type="fixed">
+  <joint name="robot2_robot2_pedestal_joint" type="fixed">
     <parent link="robot2_pedestal_link" />
     <child link="robot2_base_link" />
-    <origin xyz="0 0 0.6" rpy="0 0 ${radians(90)}" />
+    <origin xyz="0 0 0.60" rpy="0 0 ${radians(180)}" />
   </joint>
   -->
-  <!-- Add your solution to assignment 1 here -->
 </robot>

File: urdf_basics/urdf/robot/lrmate200ic_macro.xacro (robot description, xacro)
@@ -1,9 +1,13 @@
 <?xml version="1.0" ?>
 <robot xmlns:xacro="http://wiki.ros.org/xacro">
+  <!--
   <xacro:include filename="$(find urdf_basics)/urdf/include/common_materials.xacro"/>
+  -->
   <!-- NOTE: joint_limited is not used in this file -->
-  <xacro:macro name="fanuc_lrmate200ic" params="prefix joint_limited:=false">
+  <xacro:macro name="fanuc_lrmate200ic" params="prefix">
+  <link name="${prefix}tst_link"/>
     <!-- links: main serial chain -->
-    <link name="${prefix}base_link">
+    <!--
+    <link name="robot2_base_link">
       <visual>
         <origin xyz="0 0 0" rpy="0 0 0"/>
@@ -20,158 +24,24 @@
       </collision>
     </link>
-    <link name="${prefix}link_1">
-      <visual>
-        <origin xyz="0 0 0" rpy="0 0 0"/>
-        <geometry>
-          <mesh filename="package://urdf_basics/meshes/lrmate200ic/collision/link_1.stl"/>
-        </geometry>
-        <xacro:material_fanuc_yellow />
-      </visual>
-      <collision>
-        <origin xyz="0 0 0" rpy="0 0 0"/>
-        <geometry>
-          <mesh filename="package://urdf_basics/meshes/lrmate200ic/collision/link_1.stl"/>
-        </geometry>
-      </collision>
-    </link>
-    <link name="${prefix}link_2">
-      <visual>
-        <origin xyz="0 0 0" rpy="0 0 0"/>
-        <geometry>
-          <mesh filename="package://urdf_basics/meshes/lrmate200ic/collision/link_2.stl"/>
-        </geometry>
-        <xacro:material_fanuc_yellow />
-      </visual>
-      <collision>
-        <origin xyz="0 0 0" rpy="0 0 0"/>
-        <geometry>
-          <mesh filename="package://urdf_basics/meshes/lrmate200ic/collision/link_2.stl"/>
-        </geometry>
-      </collision>
-    </link>
-    <link name="${prefix}link_3">
-      <visual>
-        <origin xyz="0 0 0" rpy="0 0 0"/>
-        <geometry>
-          <mesh filename="package://urdf_basics/meshes/lrmate200ic/collision/link_3.stl"/>
-        </geometry>
-        <xacro:material_fanuc_yellow />
-      </visual>
-      <collision>
-        <origin xyz="0 0 0" rpy="0 0 0"/>
-        <geometry>
-          <mesh filename="package://urdf_basics/meshes/lrmate200ic/collision/link_3.stl"/>
-        </geometry>
-      </collision>
-    </link>
-    <link name="${prefix}link_4">
-      <visual>
-        <origin xyz="0 0 0" rpy="0 0 0"/>
-        <geometry>
-          <mesh filename="package://urdf_basics/meshes/lrmate200ic/collision/link_4.stl"/>
-        </geometry>
-        <xacro:material_fanuc_yellow />
-      </visual>
-      <collision>
-        <origin xyz="0 0 0" rpy="0 0 0"/>
-        <geometry>
-          <mesh filename="package://urdf_basics/meshes/lrmate200ic/collision/link_4.stl"/>
-        </geometry>
-      </collision>
-    </link>
-    <link name="${prefix}link_5">
-      <visual>
-        <origin xyz="0 0 0" rpy="0 0 0"/>
-        <geometry>
-          <mesh filename="package://urdf_basics/meshes/lrmate200ic/collision/link_5.stl"/>
-        </geometry>
-        <xacro:material_fanuc_yellow />
-      </visual>
-      <collision>
-        <origin xyz="0 0 0" rpy="0 0 0"/>
-        <geometry>
-          <mesh filename="package://urdf_basics/meshes/lrmate200ic/collision/link_5.stl"/>
-        </geometry>
-      </collision>
-    </link>
-    <link name="${prefix}link_6">
-      <visual>
-        <origin xyz="0 0 0" rpy="0 0 0"/>
-        <geometry>
-          <mesh filename="package://urdf_basics/meshes/lrmate200ic/collision/link_6.stl"/>
-        </geometry>
-        <xacro:material_fanuc_black />
-      </visual>
-      <collision>
-        <origin xyz="0 0 0" rpy="0 0 0"/>
-        <geometry>
-          <mesh filename="package://urdf_basics/meshes/lrmate200ic/collision/link_6.stl"/>
-        </geometry>
-      </collision>
-    </link>
+    -->
+    <!-- ROS-Industrial 'base' frame: base_link to Fanuc World Coordinates transform -->
+    <!--
+    <link name="robot2_base" />
+    <joint name="robot2_base_link-base" type="fixed">
+      <origin xyz="0 0 0.330" rpy="0 0 0"/>
+      <parent link="robot2_base_link"/>
+      <child link="robot2_base"/>
+    </joint>
+    -->
     <!-- joints: main serial chain -->
-    <joint name="${prefix}joint_1" type="revolute">
+    <!--
+    <joint name="robot2_joint_1" type="revolute">
       <origin xyz="0 0 0.330" rpy="0 0 0" />
-      <parent link="${prefix}base_link" />
-      <child link="${prefix}link_1" />
+      <parent link="robot2_base_link" />
+      <child link="robot2_link_1" />
       <axis xyz="0 0 1" />
       <limit effort="0" lower="-2.9671" upper="2.9671" velocity="6.1087" />
     </joint>
-    <joint name="${prefix}joint_2" type="revolute">
-      <origin xyz="0.075 0 0" rpy="0 0 0" />
-      <parent link="${prefix}link_1" />
-      <child link="${prefix}link_2" />
-      <axis xyz="0 1 0" />
-      <limit effort="0" lower="-1.0472" upper="2.4435" velocity="6.1087" />
-    </joint>
-    <joint name="${prefix}joint_3" type="revolute">
-      <origin xyz="0 0 0.300" rpy="0 0 0" />
-      <parent link="${prefix}link_2" />
-      <child link="${prefix}link_3" />
-      <axis xyz="0 -1 0" />
-      <limit effort="0" lower="-2.4784" upper="4.0143" velocity="6.9813" />
-    </joint>
-    <joint name="${prefix}joint_4" type="revolute">
-      <origin xyz="0 0 0.075" rpy="0 0 0"/>
-      <parent link="${prefix}link_3"/>
-      <child link="${prefix}link_4"/>
-      <axis xyz="-1 0 0"/>
-      <limit effort="0" lower="-3.3161" upper="3.3161" velocity="7.8540" />
-    </joint>
-    <joint name="${prefix}joint_5" type="revolute">
-      <origin xyz="0.320 0 0" rpy="0 0 0"/>
-      <parent link="${prefix}link_4"/>
-      <child link="${prefix}link_5"/>
-      <axis xyz="0 -1 0"/>
-      <limit effort="0" lower="-2.0944" upper="2.0944" velocity="7.8540" />
-    </joint>
-    <joint name="${prefix}joint_6" type="revolute">
-      <origin xyz="0.080 0 0" rpy="0 0 0"/>
-      <parent link="${prefix}link_5"/>
-      <child link="${prefix}link_6"/>
-      <axis xyz="-1 0 0"/>
-      <limit effort="0" lower="-6.2832" upper="6.2832" velocity="12.5664" />
-    </joint>
-    <!-- ROS-Industrial 'base' frame: base_link to Fanuc World Coordinates transform -->
-    <link name="${prefix}base" />
-    <joint name="${prefix}base_link-base" type="fixed">
-      <origin xyz="0 0 0.330" rpy="0 0 0"/>
-      <parent link="${prefix}base_link"/>
-      <child link="${prefix}base"/>
-    </joint>
-    <!-- ROS-Industrial 'flange' frame: attachment point for EEF models -->
-    <link name="${prefix}flange" />
-    <joint name="${prefix}joint_6-flange" type="fixed">
-      <origin xyz="0 0 0" rpy="0 0 0" />
-      <parent link="${prefix}link_6" />
-      <child link="${prefix}flange" />
-    </joint>
-    <!-- ROS-Industrial 'tool0' frame: all-zeros tool frame -->
-    <link name="${prefix}tool0" />
-    <joint name="${prefix}link_6-tool0" type="fixed">
-      <origin xyz="0 0 0" rpy="${pi} ${-pi/2.0} 0" />
-      <parent link="${prefix}link_6" />
-      <child link="${prefix}tool0" />
-    </joint>
-  </xacro:macro>
+    -->
+</xacro:macro>
 </robot>

Commit message: 20241118

File: urdf_basics/urdf/assignment1.xacro (robot description, xacro)
@@ -12,5 +12,5 @@
   </xacro:robot_pedestal_urdf>
   <!-- Robot1 -->
-  <xacro:include filename="$(find urdf_basics)/urdf/robot/ufactory_xarm6.urdf.xacro"/>
+  <xacro:include filename="$(find ros_industrial_support)/urdf/ufactory/ufactory_xarm6.urdf.xacro"/>
   <xacro:ufactory_xarm6 prefix="robot1_" joint_limited="true"/>
   <xacro:ufactory_xarm6 prefix="robot2_" joint_limited="true"/>

File: urdf_basics/urdf/assignment2.xacro (robot description, xacro)
@@ -12,5 +12,5 @@
   </xacro:robot_pedestal_urdf>
   <!-- Robot1 -->
-  <xacro:include filename="$(find urdf_basics)/urdf/robot/ufactory_xarm6.urdf.xacro"/>
+  <xacro:include filename="$(find ros_industrial_support)/urdf/ufactory/ufactory_xarm6.urdf.xacro"/>
   <xacro:ufactory_xarm6 prefix="robot1_" joint_limited="true"/>
   <xacro:ufactory_xarm6 prefix="robot2_" joint_limited="true"/>

File: urdf_basics/urdf/assignment3.xacro (robot description, xacro)
@@ -12,5 +12,5 @@
   </xacro:robot_pedestal_urdf>
    <!-- Robot1 -->
-  <xacro:include filename="$(find urdf_basics)/urdf/robot/ufactory_xarm6.urdf.xacro"/>
+  <xacro:include filename="$(find ros_industrial_support)/urdf/ufactory/ufactory_xarm6.urdf.xacro"/>
   <xacro:ufactory_xarm6 prefix="robot1_" joint_limited="true"/>
   <!-- Vacuum Gripper1 -->
@@ -65,6 +65,6 @@
   </joint>
   <!-- Update the below block for assignment 3 here -->
-  <xacro:include filename="$(find urdf_basics)/urdf/robot/lrmate200ic_macro.xacro"/>
-  <xacro:fanuc_lrmate200ic prefix="robot2_"/>
+  <xacro:include filename="$(find urdf_basics)/urdf/robot/lrmate200ic.urdf.xacro"/>
+  <xacro:fanuc_lrmate200ic prefix=""/>
   <!--
   <joint name="robot2_robot2_pedestal_joint" type="fixed">
@@ -74,3 +74,9 @@
   </joint>
   -->
+  <!-- robot1 to pedestal. -->
+  <joint name="robot2_to_pedestal" type="fixed">
+    <origin xyz="0 0 0.6" rpy="0 0 ${radians(90)}" />
+    <parent link="robot2_pedestal_link" />
+    <child link="base_link" />
+  </joint>
 </robot>
