Commit message: 20241118-2

File: urdf_basics/urdf/assignment1.xacro (robot description, xacro)
@@ -38,9 +38,9 @@
     <origin xyz="0 0 0.95" rpy="0 0 ${radians(90)}" />
     <parent link="robot1_pedestal_link" />
-    <child link="robot1_xarm_link" />
+    <child link="robot1_base_link" />
   </joint>
   <!-- gripper1 to robot1. -->
   <joint name="gripper1_to_robot1" type="fixed">
-    <parent link="robot1_link6" />
+    <parent link="robot1_tool_link" />
     <child link="vacuum_gripper1_base_link" />
   </joint>
@@ -77,9 +77,9 @@
     <origin xyz="0 0 0.6" rpy="0 0 ${radians(180)}" />
     <parent link="robot2_pedestal_link" />
-    <child link="robot2_xarm_link" />
+    <child link="robot2_base_link" />
   </joint>
   <!-- gripper2 to robot1. -->
   <joint name="gripper2_to_robot2" type="fixed">
-    <parent link="robot2_link6" />
+    <parent link="robot2_tool_link" />
     <child link="vacuum_gripper2_base_link" />
   </joint>

File: urdf_basics/urdf/assignment2.xacro (robot description, xacro)
@@ -38,9 +38,9 @@
     <origin xyz="0 0 0.95" rpy="0 0 ${radians(90)}" />
     <parent link="robot1_pedestal_link" />
-    <child link="robot1_xarm_link" />
+    <child link="robot1_base_link" />
   </joint>
   <!-- gripper1 to robot1. -->
   <joint name="gripper1_to_robot1" type="fixed">
-    <parent link="robot1_link6" />
+    <parent link="robot1_tool_link" />
     <child link="vacuum_gripper1_base_link" />
   </joint>
@@ -77,9 +77,9 @@
     <origin xyz="0 0 0.6" rpy="0 0 ${radians(180)}" />
     <parent link="robot2_pedestal_link" />
-    <child link="robot2_xarm_link" />
+    <child link="robot2_base_link" />
   </joint>
   <!-- gripper2 to robot1. -->
   <joint name="gripper2_to_robot2" type="fixed">
-    <parent link="robot2_link6" />
+    <parent link="robot2_tool_link" />
     <child link="vacuum_gripper2_base_link" />
   </joint>

File: urdf_basics/urdf/assignment3.xacro (robot description, xacro)
@@ -11,5 +11,5 @@
     <origin xyz="0.5 1.8 0.0" rpy="0 0 0"/>
   </xacro:robot_pedestal_urdf>
-   <!-- Robot1 -->
+  <!-- Robot1 -->
   <xacro:include filename="$(find ros_industrial_support)/urdf/ufactory/ufactory_xarm6.urdf.xacro"/>
   <xacro:ufactory_xarm6 prefix="robot1_" joint_limited="true"/>
@@ -20,4 +20,5 @@
   <xacro:include filename="$(find ros_industrial_support)/urdf/bin/bin.urdf.xacro"/>
   <xacro:bin_urdf prefix="bin_1_"/>
+  <xacro:bin_urdf prefix="bin_2_"/>
   <!-- Joints -->
   <joint name="world_interface_to_world" type="fixed">
@@ -35,9 +36,9 @@
     <origin xyz="0 0 0.95" rpy="0 0 ${radians(90)}" />
     <parent link="robot1_pedestal_link" />
-    <child link="robot1_xarm_link" />
+    <child link="robot1_base_link" />
   </joint>
   <!-- gripper1 to robot1. -->
   <joint name="gripper1_to_robot1" type="fixed">
-    <parent link="robot1_link6" />
+    <parent link="robot1_tool_link" />
     <child link="vacuum_gripper1_base_link" />
   </joint>
@@ -47,4 +48,10 @@
     <child link="bin_1_base_link" />
     <origin xyz="-8.0 -2.2 0" rpy="0 0 0" />
+  </joint>
+  <!-- bin 2 -->
+  <joint name="bin_2_joint" type="fixed">
+    <parent link="world_interface" />
+    <child link="bin_2_base_link" />
+    <origin xyz="2.5 1.8 0" rpy="0 0 0" />
   </joint>
   <link name="robot2_pedestal_link">
@@ -66,5 +73,5 @@
   <!-- Update the below block for assignment 3 here -->
   <xacro:include filename="$(find urdf_basics)/urdf/robot/lrmate200ic.urdf.xacro"/>
-  <xacro:fanuc_lrmate200ic prefix=""/>
+  <xacro:fanuc_lrmate200ic prefix="robot2_"/>
   <!--
   <joint name="robot2_robot2_pedestal_joint" type="fixed">
@@ -75,4 +82,5 @@
   -->
   <!-- robot1 to pedestal. -->
+  <!--
   <joint name="robot2_to_pedestal" type="fixed">
     <origin xyz="0 0 0.6" rpy="0 0 ${radians(90)}" />
@@ -80,3 +88,4 @@
     <child link="base_link" />
   </joint>
+  -->
 </robot>

File: urdf_basics/urdf/robot/lrmate200ic.urdf.xacro (robot description, xacro)
@@ -1,10 +1,10 @@
 <?xml version="1.0" ?>
 <robot xmlns:xacro="http://wiki.ros.org/xacro">
+  <xacro:include filename="$(find urdf_basics)/urdf/include/common_materials.xacro"/>
+  <!-- NOTE: joint_limited is not used in this file -->
+  <xacro:macro name="fanuc_lrmate200ic" params="prefix joint_limited:=false">
   <!--
-  <xacro:include filename="$(find urdf_basics)/urdf/include/common_materials.xacro"/>
+  <link name="${prefix}tst_link"/>
   -->
-  <!-- NOTE: joint_limited is not used in this file -->
-  <xacro:macro name="fanuc_lrmate200ic" params="prefix">
-  <link name="${prefix}tst_link"/>
     <!-- links: main serial chain -->
     <!--
@@ -16,5 +16,5 @@
         </geometry>
         <xacro:material_fanuc_gray24 />
-      </visual>
+        </visual>
       <collision>
         <origin xyz="0 0 0" rpy="0 0 0"/>
@@ -44,4 +44,4 @@
     </joint>
     -->
-</xacro:macro>
+  </xacro:macro>
 </robot>
