Commit message: 20241119

File: urdf_basics/urdf/assignment3.urdf.xacro (robot description, xacro)
@@ -66,5 +66,5 @@
     </visual>
   </link>
-  <joint name="robot2_pedestal_joint" type="fixed">
+  <joint name="robot2_pedestal_joint_to_world" type="fixed">
     <origin xyz="-7.8 -1.5 0" />
     <parent link="world" />
@@ -74,18 +74,16 @@
   <xacro:include filename="$(find urdf_basics)/urdf/robot/lrmate200ic.urdf.xacro"/>
   <xacro:fanuc_lrmate200ic prefix="robot2_"/>
-  <!--
-  <joint name="robot2_robot2_pedestal_joint" type="fixed">
-    <parent link="robot2_pedestal_link" />
-    <child link="robot2_base_link" />
-    <origin xyz="0 0 0.60" rpy="0 0 ${radians(180)}" />
-  </joint>
-  -->
-  <!-- robot1 to pedestal. -->
-  <!--
+  <!-- robot2 to pedestal. -->
   <joint name="robot2_to_pedestal" type="fixed">
     <origin xyz="0 0 0.6" rpy="0 0 ${radians(90)}" />
     <parent link="robot2_pedestal_link" />
-    <child link="base_link" />
+    <child link="robot2_base_link" />
   </joint>
-  -->
+  <!-- Vacuum Gripper2 -->
+  <xacro:vacuum_gripper_urdf prefix="vacuum_gripper2_" joint_prefix="vacuum_gripper2_joint"/>
+  <!-- gripper2 to robot1. -->
+  <joint name="gripper2_to_robot2" type="fixed">
+    <parent link="robot2_tool_link" />
+    <child link="vacuum_gripper2_base_link" />
+  </joint>
 </robot>

File: urdf_basics/urdf/robot/lrmate200ic.urdf.xacro (robot description, xacro)
@@ -4,10 +4,5 @@
   <!-- NOTE: joint_limited is not used in this file -->
   <xacro:macro name="fanuc_lrmate200ic" params="prefix joint_limited:=false">
-  <!--
-  <link name="${prefix}tst_link"/>
-  -->
-    <!-- links: main serial chain -->
-    <!--
-    <link name="robot2_base_link">
+    <link name="${prefix}base_link">
       <visual>
         <origin xyz="0 0 0" rpy="0 0 0"/>
@@ -16,5 +11,5 @@
         </geometry>
         <xacro:material_fanuc_gray24 />
-        </visual>
+      </visual>
       <collision>
         <origin xyz="0 0 0" rpy="0 0 0"/>
@@ -24,24 +19,142 @@
       </collision>
     </link>
-    -->
-    <!-- ROS-Industrial 'base' frame: base_link to Fanuc World Coordinates transform -->
-    <!--
-    <link name="robot2_base" />
-    <joint name="robot2_base_link-base" type="fixed">
-      <origin xyz="0 0 0.330" rpy="0 0 0"/>
-      <parent link="robot2_base_link"/>
-      <child link="robot2_base"/>
-    </joint>
-    -->
-    <!-- joints: main serial chain -->
-    <!--
-    <joint name="robot2_joint_1" type="revolute">
+    <link name="${prefix}link_1">
+      <visual>
+        <origin xyz="0 0 0" rpy="0 0 0"/>
+        <geometry>
+          <mesh filename="package://urdf_basics/meshes/lrmate200ic/collision/link_1.stl"/>
+        </geometry>
+        <xacro:material_fanuc_yellow />
+      </visual>
+      <collision>
+        <origin xyz="0 0 0" rpy="0 0 0"/>
+        <geometry>
+          <mesh filename="package://urdf_basics/meshes/lrmate200ic/collision/link_1.stl"/>
+        </geometry>
+      </collision>
+    </link>
+    <link name="${prefix}link_2">
+      <visual>
+        <origin xyz="0 0 0" rpy="0 0 0"/>
+        <geometry>
+          <mesh filename="package://urdf_basics/meshes/lrmate200ic/collision/link_2.stl"/>
+        </geometry>
+        <xacro:material_fanuc_yellow />
+      </visual>
+      <collision>
+        <origin xyz="0 0 0" rpy="0 0 0"/>
+        <geometry>
+          <mesh filename="package://urdf_basics/meshes/lrmate200ic/collision/link_2.stl"/>
+        </geometry>
+      </collision>
+    </link>
+    <link name="${prefix}link_3">
+      <visual>
+        <origin xyz="0 0 0" rpy="0 0 0"/>
+        <geometry>
+          <mesh filename="package://urdf_basics/meshes/lrmate200ic/collision/link_3.stl"/>
+        </geometry>
+        <xacro:material_fanuc_yellow />
+      </visual>
+      <collision>
+        <origin xyz="0 0 0" rpy="0 0 0"/>
+        <geometry>
+          <mesh filename="package://urdf_basics/meshes/lrmate200ic/collision/link_3.stl"/>
+        </geometry>
+      </collision>
+    </link>
+    <link name="${prefix}link_4">
+      <visual>
+        <origin xyz="0 0 0" rpy="0 0 0"/>
+        <geometry>
+          <mesh filename="package://urdf_basics/meshes/lrmate200ic/collision/link_4.stl"/>
+        </geometry>
+        <xacro:material_fanuc_yellow />
+      </visual>
+      <collision>
+        <origin xyz="0 0 0" rpy="0 0 0"/>
+        <geometry>
+          <mesh filename="package://urdf_basics/meshes/lrmate200ic/collision/link_4.stl"/>
+        </geometry>
+      </collision>
+    </link>
+    <link name="${prefix}link_5">
+      <visual>
+        <origin xyz="0 0 0" rpy="0 0 0"/>
+        <geometry>
+          <mesh filename="package://urdf_basics/meshes/lrmate200ic/collision/link_5.stl"/>
+        </geometry>
+        <xacro:material_fanuc_yellow />
+      </visual>
+      <collision>
+        <origin xyz="0 0 0" rpy="0 0 0"/>
+        <geometry>
+          <mesh filename="package://urdf_basics/meshes/lrmate200ic/collision/link_5.stl"/>
+        </geometry>
+      </collision>
+    </link>
+    <link name="${prefix}link_6">
+      <visual>
+        <origin xyz="0 0 0" rpy="0 0 0"/>
+        <geometry>
+          <mesh filename="package://urdf_basics/meshes/lrmate200ic/collision/link_6.stl"/>
+        </geometry>
+        <xacro:material_fanuc_black />
+      </visual>
+      <collision>
+        <origin xyz="0 0 0" rpy="0 0 0"/>
+        <geometry>
+          <mesh filename="package://urdf_basics/meshes/lrmate200ic/collision/link_6.stl"/>
+        </geometry>
+      </collision>
+    </link>
+    <joint name="${prefix}joint_1" type="revolute">
       <origin xyz="0 0 0.330" rpy="0 0 0" />
-      <parent link="robot2_base_link" />
-      <child link="robot2_link_1" />
+      <parent link="${prefix}base_link" />
+      <child link="${prefix}link_1" />
       <axis xyz="0 0 1" />
       <limit effort="0" lower="-2.9671" upper="2.9671" velocity="6.1087" />
     </joint>
-    -->
+    <joint name="${prefix}joint_2" type="revolute">
+      <origin xyz="0.075 0 0" rpy="0 0 0" />
+      <parent link="${prefix}link_1" />
+      <child link="${prefix}link_2" />
+      <axis xyz="0 1 0" />
+      <limit effort="0" lower="-1.0472" upper="2.4435" velocity="6.1087" />
+    </joint>
+    <joint name="${prefix}joint_3" type="revolute">
+      <origin xyz="0 0 0.300" rpy="0 0 0" />
+      <parent link="${prefix}link_2" />
+      <child link="${prefix}link_3" />
+      <axis xyz="0 -1 0" />
+      <limit effort="0" lower="-2.4784" upper="4.0143" velocity="6.9813" />
+    </joint>
+    <joint name="${prefix}joint_4" type="revolute">
+      <origin xyz="0 0 0.075" rpy="0 0 0"/>
+      <parent link="${prefix}link_3"/>
+      <child link="${prefix}link_4"/>
+      <axis xyz="-1 0 0"/>
+      <limit effort="0" lower="-3.3161" upper="3.3161" velocity="7.8540" />
+    </joint>
+    <joint name="${prefix}joint_5" type="revolute">
+      <origin xyz="0.320 0 0" rpy="0 0 0"/>
+      <parent link="${prefix}link_4"/>
+      <child link="${prefix}link_5"/>
+      <axis xyz="0 -1 0"/>
+      <limit effort="0" lower="-2.0944" upper="2.0944" velocity="7.8540" />
+    </joint>
+    <joint name="${prefix}joint_6" type="revolute">
+      <origin xyz="0.080 0 0" rpy="0 0 0"/>
+      <parent link="${prefix}link_5"/>
+      <child link="${prefix}link_6"/>
+      <axis xyz="-1 0 0"/>
+      <limit effort="0" lower="-6.2832" upper="6.2832" velocity="12.5664" />
+    </joint>
+  <link name="${prefix}tool_link"/>
+  <joint name="${prefix}link_6_eff" type="fixed">
+    <origin xyz="0 0 0" rpy="${pi} ${-pi/2.0} 0" />
+    <parent link="${prefix}link_6" />
+    <child link="${prefix}tool_link" />
+  </joint>
   </xacro:macro>
 </robot>

File: urdf_basics/urdf/robot/lrmate200ic_environment.urdf.xacro (robot description, xacro)
@@ -1,5 +1,5 @@
 <?xml version="1.0" ?>
 <robot name="fanuc_lrmate200ic" xmlns:xacro="http://wiki.ros.org/xacro">
-  <xacro:include filename="$(find urdf_basics)/urdf/robot/lrmate200ic_macro.xacro"/>
+  <xacro:include filename="$(find urdf_basics)/urdf/robot/lrmate200ic.urdf.xacro"/>
   <xacro:fanuc_lrmate200ic prefix=""/>
 </robot>
